Commit message: add camera and marker to robot description

File: f1tenth_description/urdf/const.xacro (robot description, xacro)
@@ -4,4 +4,8 @@
     <xacro:arg name="robot_name" default="f1tenth"/>
     <xacro:property name="robot_name" value="$(arg robot_name)" />
+    <xacro:arg name="add_camera" default="false"/>
+    <xacro:property name="add_camera" value="$(arg add_camera)" />
+    <xacro:arg name="add_aruco" default="false"/>
+    <xacro:property name="add_aruco" value="$(arg add_aruco)" />
     <!-- <xacro:property name="params_path" value="$(arg params_path)"/> -->
     <!-- Wheels -->

File: f1tenth_description/urdf/joints.xacro (robot description, xacro)
@@ -7,6 +7,6 @@
         <axis xyz="0 0 1" />
         <limit lower="-0.6" upper="+0.6"
-               velocity="1.0" effort="25" />
-        <origin xyz="0.1575 0.1025 0.055" rpy="0 0 0"/>
+            velocity="1.0" effort="25" />
+        <origin xyz="0.1575 0.1025 0.055" rpy="0 0 0" />
     </joint>
     <joint name="front_right_wheel_steering_joint" type="revolute">
@@ -15,6 +15,6 @@
         <axis xyz="0 0 1" />
         <limit lower="-0.6" upper="+0.6"
-               velocity="1.0" effort="25" />
-        <origin xyz="0.1575 -0.1025 0.055" rpy="0 0 0"/>
+            velocity="1.0" effort="25" />
+        <origin xyz="0.1575 -0.1025 0.055" rpy="0 0 0" />
     </joint>
     <!-- Drive joints -->
@@ -33,5 +33,5 @@
         <parent link="base_link" />
         <axis xyz="0 1 0" />
-        <origin xyz="-0.1575 0.1025 0.055" rpy="0 0 0"/>
+        <origin xyz="-0.1575 0.1025 0.055" rpy="0 0 0" />
     </joint>
     <joint name="rear_right_wheel_joint" type="continuous">
@@ -39,5 +39,5 @@
         <parent link="base_link" />
         <axis xyz="0 1 0" />
-        <origin xyz="-0.1575 -0.1025 0.055" rpy="0 0 0"/>
+        <origin xyz="-0.1575 -0.1025 0.055" rpy="0 0 0" />
     </joint>
     <!-- Chassis Joints-->
@@ -45,10 +45,10 @@
         <child link="box_visual" />
         <parent link="base_link" />
-        <origin xyz="-0.1554 0.09 0.2" rpy="0 0 0"/>
+        <origin xyz="-0.1554 0.09 0.2" rpy="0 0 0" />
     </joint>
     <joint name="base_link_to_lower_chassis" type="fixed">
         <child link="lower_chassis" />
         <parent link="base_link" />
-        <origin xyz="-0.155 0.09 0.055" rpy="0 0 0"/>
+        <origin xyz="-0.155 0.09 0.055" rpy="0 0 0" />
     </joint>
     <!-- Sensor Joints -->
@@ -56,5 +56,14 @@
         <child link="hokuyo_10lx_lidar_link" />
         <parent link="base_link" />
-        <origin xyz="0.1 0 0.15" rpy="0 0 0"/>
+        <origin xyz="0.1 0 0.15" rpy="0 0 0" />
     </joint>
+    <xacro:if value="${add_aruco}">
+        <gazebo>
+            <joint name="aruco_marker_joint" type="fixed">
+                <pose relative_to="box_visual">0 0 0 0 0 0</pose>
+                <child>aruco_link</child>
+                <parent>box_visual</parent>
+            </joint>
+        </gazebo>
+    </xacro:if>
 </robot>

File: f1tenth_description/urdf/links.xacro (robot description, xacro)
@@ -41,3 +41,8 @@
       <origin xyz="0 0 0" rpy="0 0 0"/>
     </xacro:cylinder_link_nomesh>
+    <!-- AruCo marker -->
+    <xacro:if value="${add_aruco}">
+        <xacro:include filename="$(find f1tenth_description)/sdf/aruco_marker/model.urdf.xacro" />
+        <xacro:aruco_marker xyz="-0.20 0 0.183" rpy="0 0 0"/>
+    </xacro:if>
 </robot>

File: f1tenth_description/urdf/robot.urdf.xacro (robot description, xacro)
@@ -8,4 +8,5 @@
     <xacro:include filename="$(find f1tenth_description)/urdf/links.xacro" />
     <xacro:include filename="$(find f1tenth_description)/urdf/joints.xacro" />
+    <xacro:include filename="$(find f1tenth_description)/urdf/d435.xacro" />
     <!-- Gazebo stuff -->
     <xacro:include filename="$(find f1tenth_description)/gazebo/ackermann.gazebo.xacro" />

Commit message: take camera name in macro

File: f1tenth_description/urdf/const.xacro (robot description, xacro)
@@ -4,4 +4,6 @@
     <xacro:arg name="robot_name" default="f1tenth"/>
     <xacro:property name="robot_name" value="$(arg robot_name)" />
+    <xacro:arg name="camera_name" default="d435"/>
+    <xacro:property name="camera_name" value="$(arg camera_name)" />
     <xacro:arg name="add_camera" default="false"/>
     <xacro:property name="add_camera" value="$(arg add_camera)" />

File: f1tenth_description/urdf/d435.xacro (robot description, xacro)
@@ -4,5 +4,5 @@
   <xacro:include filename="$(find realsense2_description)/urdf/_d435.urdf.xacro" />
   <xacro:if value="${add_camera}">
-    <xacro:sensor_d435 gazebo="true" name="d435" parent="base_link"
+    <xacro:sensor_d435 gazebo="true" name="${camera_name}" parent="base_link"
       use_nominal_extrinsics="true"
       enable_infra1="false" enable_infra2="false" enable_color="true" enable_depth="true"

File: f1tenth_description/urdf/joints.xacro (robot description, xacro)
@@ -58,4 +58,5 @@
         <origin xyz="0.1 0 0.15" rpy="0 0 0" />
     </joint>
+    <!-- Add AruCo marker  -->
     <xacro:if value="${add_aruco}">
         <gazebo>
